Commit message: Update 01/06

File: src/my_project/urdf/robot.gazebo.xacro (robot description, xacro)
@@ -102,5 +102,5 @@
     </plugin>
   </gazebo>
-  <!--gazebo reference="sonar1_link">
+  <gazebo reference="sonar1_link">
    <sensor type="ray" name="head_hokuyo_sensor1">
      <pose>0 0 0 0 0 0</pose>
@@ -128,5 +128,5 @@
      </ray>
      <plugin name="gazebo_ros_head_hokuyo_controller" filename="libgazebo_ros_laser.so">
-       <topicName>/my_turtlebot/sonar1</topicName>
+       <topicName>/my_project/sonar1</topicName>
        <frameName>sonar1_link</frameName>
      </plugin>
@@ -159,5 +159,5 @@
     </ray>
     <plugin name="gazebo_ros_head_hokuyo_controller" filename="libgazebo_ros_laser.so">
-      <topicName>/my_turtlebot/sonar2</topicName>
+      <topicName>/my_project/sonar2</topicName>
       <frameName>sonar2_link</frameName>
     </plugin>
@@ -190,8 +190,39 @@
      </ray>
      <plugin name="gazebo_ros_head_hokuyo_controller" filename="libgazebo_ros_laser.so">
-       <topicName>/my_turtlebot/sonar3</topicName>
+       <topicName>/my_project/sonar3</topicName>
        <frameName>sonar3_link</frameName>
      </plugin>
    </sensor>
- </gazebo-->
+ </gazebo>
+ <gazebo reference="sonar4_link">
+  <sensor type="ray" name="head_hokuyo_sensor4">
+    <pose>0 0 0 0 0 0</pose>
+    <visualize>true</visualize>
+    <update_rate>40</update_rate>
+    <ray>
+      <scan>
+        <horizontal>
+          <samples>720</samples>
+          <resolution>1</resolution>
+          <min_angle>-0.436332</min_angle>
+          <max_angle>0.436332</max_angle>
+        </horizontal>
+      </scan>
+      <range>
+        <min>0.04</min>
+        <max>0.3</max>
+        <resolution>0.01</resolution>
+      </range>
+      <noise>
+        <type>gaussian</type>
+        <mean>0.0</mean>
+        <stddev>0.01</stddev>
+      </noise>
+    </ray>
+    <plugin name="gazebo_ros_head_hokuyo_controller" filename="libgazebo_ros_laser.so">
+      <topicName>/my_project/sonar4</topicName>
+      <frameName>sonar4_link</frameName>
+    </plugin>
+  </sensor>
+</gazebo>
 </robot>

File: src/my_project/urdf/robot.urdf.xacro (robot description, xacro)
@@ -10,8 +10,9 @@
   </joint>
   <link name="base_link">
-    <pose>0 0 0.07 0 0 0</pose>
+    <pose>0 0 0 0 0 0</pose>
     <visual>
-      <geometry>
-        <mesh filename="package://my_project/meshes/bases/burger_base.stl" scale="0.001 0.001 0.001"/>
+      <origin xyz="0.06 0.006 -0.3" rpy="0 0 -1.5708" />
+      <geometry>
+        <mesh filename="package://my_project/meshes/bases/Base.stl" scale="0.001 0.001 0.001"/>
       </geometry>
       <material name="light_black"/>
@@ -32,5 +33,5 @@
     <parent link="base_link"/>
     <child link="wheel_left_link"/>
-    <origin xyz="0 0.17 -0.3" rpy="-1.57 0 0"/>
+    <origin xyz="0.027 0.17 -0.3" rpy="-1.57 0 0"/>
     <axis xyz="0 0 1"/>
   </joint>
@@ -70,5 +71,5 @@
     <parent link="base_link"/>
     <child link="wheel_right_link"/>
-    <origin xyz="0.0 -0.17 -0.3" rpy="-1.57 0 0"/>
+    <origin xyz="0.027 -0.17 -0.3" rpy="-1.57 0 0"/>
     <axis xyz="0 0 1"/>
   </joint>
@@ -173,5 +174,5 @@
     <parent link="base_link"/>
     <child link="sonar1_link" />
-    <origin xyz="0.15 0 -0.25" rpy="0 0 1.0472"/>
+    <origin xyz="0.11780 0.11780 -0.25" rpy="0 0 0.7853"/>
   </joint>
   <link name="sonar1_link">
@@ -180,5 +181,5 @@
     <parent link="base_link"/>
     <child link="sonar2_link" />
-    <origin xyz="0.15 0 -0.25" rpy="0 0 -1.0472"/>
+    <origin xyz="0.11780 -0.11780 -0.25" rpy="0 0 -0.7853"/>
   </joint>
   <link name="sonar2_link">
@@ -187,7 +188,14 @@
     <parent link="base_link"/>
     <child link="sonar3_link" />
-    <origin xyz="-0.15 0 -0.25" rpy="0 0 2.61799"/>
+    <origin xyz="-0.11780 0.11780 -0.25" rpy="0 0 2.35619"/>
   </joint>
   <link name="sonar3_link">
   </link>
+  <joint name="sonar4_joint" type="fixed">
+    <parent link="base_link"/>
+    <child link="sonar4_link" />
+    <origin xyz="-0.11780 -0.11780 -0.25" rpy="0 0 -2.35619"/>
+  </joint>
+  <link name="sonar4_link">
+  </link>
 </robot>

Commit message: Update 14 August

File: src/my_project/urdf/robot.gazebo.xacro (robot description, xacro)
@@ -3,25 +3,25 @@
   <xacro:arg name="camera_visual" default="false"/>
   <gazebo reference="base_link">
-    <material>Gazebo/DarkGrey</material>
+    <material>Gazebo/Motorway</material>
   </gazebo>
   <gazebo reference="wheel_left_link">
     <mu1>0.5</mu1>
     <mu2>0.5</mu2>
-    <kp>500000.0</kp>
+    <kp>5000000.0</kp>
     <kd>10.0</kd>
     <minDepth>0.001</minDepth>
-    <maxVel>0.1</maxVel>
+    <maxVel>0.5</maxVel>
     <fdir1>1 0 0</fdir1>
-    <material>Gazebo/FlatBlack</material>
+    <material>Gazebo/Black</material>
   </gazebo>
   <gazebo reference="wheel_right_link">
     <mu1>0.5</mu1>
     <mu2>0.5</mu2>
-    <kp>500000.0</kp>
+    <kp>5000000.0</kp>
     <kd>10.0</kd>
     <minDepth>0.001</minDepth>
-    <maxVel>0.1</maxVel>
+    <maxVel>0.5</maxVel>
     <fdir1>1 0 0</fdir1>
-    <material>Gazebo/FlatBlack</material>
+    <material>Gazebo/Black</material>
   </gazebo>
   <gazebo reference="caster_back_link">

File: src/my_project/urdf/robot.urdf.xacro (robot description, xacro)
@@ -33,5 +33,5 @@
     <parent link="base_link"/>
     <child link="wheel_left_link"/>
-    <origin xyz="0.027 0.17 -0.3" rpy="-1.57 0 0"/>
+    <origin xyz="0.013 0.17 -0.3" rpy="-1.57 0 0"/>
     <axis xyz="0 0 1"/>
   </joint>
@@ -65,5 +65,5 @@
     <actuator name="wheel_left_motor">
       <hardwareInterface>VelocityJointInterface</hardwareInterface>
-      <mechanicalReduction>1</mechanicalReduction>
+      <mechanicalReduction>34</mechanicalReduction>
     </actuator>
   </transmission>
@@ -71,5 +71,5 @@
     <parent link="base_link"/>
     <child link="wheel_right_link"/>
-    <origin xyz="0.027 -0.17 -0.3" rpy="-1.57 0 0"/>
+    <origin xyz="0.013 -0.17 -0.3" rpy="-1.57 0 0"/>
     <axis xyz="0 0 1"/>
   </joint>
@@ -103,5 +103,5 @@
     <actuator name="wheel_right_motor">
       <hardwareInterface>VelocityJointInterface</hardwareInterface>
-      <mechanicalReduction>1</mechanicalReduction>
+      <mechanicalReduction>34</mechanicalReduction>
     </actuator>
   </transmission>
