Commit message: Update 22 June

File: src/my_project/urdf/robot.urdf.xacro (robot description, xacro)
@@ -153,5 +153,5 @@
   <link name="camera_link">
     <collision>
-      <origin xyz="0.005 0.011 0.013" rpy="0 0 0"/>
+      <origin xyz="0.05 0.011 0.013" rpy="0 0 0"/>
       <geometry>
         <box size="0.015 0.030 0.027"/>

Commit message: Update 26 June

File: src/my_project/urdf/robot.urdf.xacro (robot description, xacro)
@@ -147,5 +147,5 @@
   </link>
   <joint name="camera_joint" type="fixed">
-    <origin xyz="0.040 -0.011 0.130" rpy="0 0.174 0"/>
+    <origin xyz="0.0 0.0 0.2" rpy="0 0.0 0"/>
     <parent link="base_link"/>
     <child link="camera_link"/>
@@ -153,12 +153,12 @@
   <link name="camera_link">
     <collision>
-      <origin xyz="0.05 0.011 0.013" rpy="0 0 0"/>
-      <geometry>
-        <box size="0.015 0.030 0.027"/>
+      <origin xyz="0.16 0.0 0.0" rpy="0 0 0"/>
+      <geometry>
+        <box size="0.005 0.015 0.015"/>
       </geometry>
     </collision>
   </link>
   <joint name="camera_rgb_joint" type="fixed">
-    <origin xyz="0.003 0.011 0.009" rpy="0 0 0"/>
+    <origin xyz="0.16 0.0 0.0" rpy="0 0 0"/>
     <parent link="camera_link"/>
     <child link="camera_rgb_frame"/>
@@ -166,5 +166,5 @@
   <link name="camera_rgb_frame"/>
   <joint name="camera_rgb_optical_joint" type="fixed">
-    <origin xyz="0 0 0" rpy="-1.57 0 -1.57"/>
+    <origin xyz="0.0 0 0" rpy="0 0 0"/>
     <parent link="camera_rgb_frame"/>
     <child link="camera_rgb_optical_frame"/>

Commit message: Update 04 September

File: src/my_project/urdf/robot.urdf.xacro (robot description, xacro)
@@ -38,7 +38,7 @@
   <link name="wheel_left_link">
     <visual>
-      <origin xyz="0 0 0" rpy="1.57 0 0"/>
-      <geometry>
-        <mesh filename="package://my_project/meshes/wheels/left_tire.stl" scale="0.001 0.001 0.001"/>
+      <origin xyz="0 0 0" rpy="0 0 0"/>
+      <geometry>
+        <mesh filename="package://my_project/meshes/wheels/Wheel.stl" scale="0.01 0.01 0.01"/>
       </geometry>
       <material name="dark"/>
@@ -76,7 +76,7 @@
   <link name="wheel_right_link">
     <visual>
-      <origin xyz="0 0 0" rpy="1.57 0 0"/>
-      <geometry>
-        <mesh filename="package://my_project/meshes/wheels/right_tire.stl" scale="0.001 0.001 0.001"/>
+      <origin xyz="0 0 0" rpy="0 3.1415 0"/>
+      <geometry>
+        <mesh filename="package://my_project/meshes/wheels/Wheel.stl" scale="0.01 0.01 0.01"/>
       </geometry>
       <material name="dark"/>
